File: Matrix.sch (KiCad schematic (older format))
At the start: 102 parts

Commit message: Added the new coloumn
Added all the needed components, just need to fix the PCB.
Parts:
- D1, D10, D11, D12, D13, D14, D15, D16, D17, D18, D19, D2, D20, D21, D22, D23, D24, D25, D26, D27, D28, D29, D3, D30, D31, D32, D33, D34, D35, D36, D37, D38, D39, D4, D40, D41, D42, D43, D44, D45, D46, D47, D48, D49, D5, D50, D51, D6, D7, D8, D9: footprint (none) -> Diode_SMD:D_1206_3216Metric
- MX1, MX10, MX11, MX12, MX13, MX14, MX15, MX16, MX17, MX18, MX19, MX2, MX20, MX21, MX22, MX23, MX24, MX25, MX26, MX27, MX28, MX29, MX3, MX30, MX31, MX32, MX33, MX34, MX35, MX36, MX37, MX38, MX39, MX4, MX40, MX41, MX42, MX43, MX44, MX45, MX46, MX47, MX48, MX49, MX5, MX50, MX51, MX6, MX7, MX8, MX9: footprint (none) -> footprints:Kailh_socket_MX

Commit message: Finished first revision
Should be okay to order now
Parts:
- D1, D18, D51: footprint Diode_SMD:D_1206_3216Metric -> Diode_SMD:D_SOD-123
- D10: renamed from D36; footprint Diode_SMD:D_1206_3216Metric -> Diode_SMD:D_SOD-123
- D11: renamed from D40; footprint Diode_SMD:D_1206_3216Metric -> Diode_SMD:D_SOD-123
- D12: renamed from D44; footprint Diode_SMD:D_1206_3216Metric -> Diode_SMD:D_SOD-123
- D13: renamed from D48; footprint Diode_SMD:D_1206_3216Metric -> Diode_SMD:D_SOD-123
- D14: renamed from D2; footprint Diode_SMD:D_1206_3216Metric -> Diode_SMD:D_SOD-123
- D15: renamed from D6; footprint Diode_SMD:D_1206_3216Metric -> Diode_SMD:D_SOD-123
- D16: renamed from D10; footprint Diode_SMD:D_1206_3216Metric -> Diode_SMD:D_SOD-123
- D17: renamed from D14; footprint Diode_SMD:D_1206_3216Metric -> Diode_SMD:D_SOD-123
- D19: renamed from D22; footprint Diode_SMD:D_1206_3216Metric -> Diode_SMD:D_SOD-123
- D2: renamed from D5; footprint Diode_SMD:D_1206_3216Metric -> Diode_SMD:D_SOD-123
- D20: renamed from D26; footprint Diode_SMD:D_1206_3216Metric -> Diode_SMD:D_SOD-123
- D21: renamed from D29; footprint Diode_SMD:D_1206_3216Metric -> Diode_SMD:D_SOD-123
- D22: renamed from D33; footprint Diode_SMD:D_1206_3216Metric -> Diode_SMD:D_SOD-123
- D23: renamed from D37; footprint Diode_SMD:D_1206_3216Metric -> Diode_SMD:D_SOD-123
- D24: renamed from D41; footprint Diode_SMD:D_1206_3216Metric -> Diode_SMD:D_SOD-123
- D25: renamed from D45; footprint Diode_SMD:D_1206_3216Metric -> Diode_SMD:D_SOD-123
- D26: renamed from D49; footprint Diode_SMD:D_1206_3216Metric -> Diode_SMD:D_SOD-123
- D27: renamed from D3; footprint Diode_SMD:D_1206_3216Metric -> Diode_SMD:D_SOD-123
- D28: renamed from D7; footprint Diode_SMD:D_1206_3216Metric -> Diode_SMD:D_SOD-123
- D29: renamed from D11; footprint Diode_SMD:D_1206_3216Metric -> Diode_SMD:D_SOD-123
- D3: renamed from D9; footprint Diode_SMD:D_1206_3216Metric -> Diode_SMD:D_SOD-123
- D30: renamed from D15; footprint Diode_SMD:D_1206_3216Metric -> Diode_SMD:D_SOD-123
- D31: renamed from D19; footprint Diode_SMD:D_1206_3216Metric -> Diode_SMD:D_SOD-123
- D32: renamed from D23; footprint Diode_SMD:D_1206_3216Metric -> Diode_SMD:D_SOD-123
- D33: renamed from D27; footprint Diode_SMD:D_1206_3216Metric -> Diode_SMD:D_SOD-123
- D34: renamed from D30; footprint Diode_SMD:D_1206_3216Metric -> Diode_SMD:D_SOD-123
- D35: renamed from D34; footprint Diode_SMD:D_1206_3216Metric -> Diode_SMD:D_SOD-123
- D36: renamed from D38; footprint Diode_SMD:D_1206_3216Metric -> Diode_SMD:D_SOD-123
- D37: renamed from D42; footprint Diode_SMD:D_1206_3216Metric -> Diode_SMD:D_SOD-123
- D38: renamed from D46; footprint Diode_SMD:D_1206_3216Metric -> Diode_SMD:D_SOD-123
- D39: renamed from D50; footprint Diode_SMD:D_1206_3216Metric -> Diode_SMD:D_SOD-123
- D4: renamed from D13; footprint Diode_SMD:D_1206_3216Metric -> Diode_SMD:D_SOD-123
- D40: renamed from D4; footprint Diode_SMD:D_1206_3216Metric -> Diode_SMD:D_SOD-123
- D41: renamed from D8; footprint Diode_SMD:D_1206_3216Metric -> Diode_SMD:D_SOD-123
- D42: renamed from D12; footprint Diode_SMD:D_1206_3216Metric -> Diode_SMD:D_SOD-123
- D43: renamed from D16; footprint Diode_SMD:D_1206_3216Metric -> Diode_SMD:D_SOD-123
- D44: renamed from D20; footprint Diode_SMD:D_1206_3216Metric -> Diode_SMD:D_SOD-123
- D45: renamed from D24; footprint Diode_SMD:D_1206_3216Metric -> Diode_SMD:D_SOD-123
- D46: renamed from D31; footprint Diode_SMD:D_1206_3216Metric -> Diode_SMD:D_SOD-123
- D47: renamed from D35; footprint Diode_SMD:D_1206_3216Metric -> Diode_SMD:D_SOD-123
- D48: renamed from D39; footprint Diode_SMD:D_1206_3216Metric -> Diode_SMD:D_SOD-123
- D49: renamed from D43; footprint Diode_SMD:D_1206_3216Metric -> Diode_SMD:D_SOD-123
- D5: renamed from D17; footprint Diode_SMD:D_1206_3216Metric -> Diode_SMD:D_SOD-123
- D50: renamed from D47; footprint Diode_SMD:D_1206_3216Metric -> Diode_SMD:D_SOD-123
- D6: renamed from D21; footprint Diode_SMD:D_1206_3216Metric -> Diode_SMD:D_SOD-123
- D7: renamed from D25; footprint Diode_SMD:D_1206_3216Metric -> Diode_SMD:D_SOD-123
- D8: renamed from D28; footprint Diode_SMD:D_1206_3216Metric -> Diode_SMD:D_SOD-123
- D9: renamed from D32; footprint Diode_SMD:D_1206_3216Metric -> Diode_SMD:D_SOD-123
- renumbered MX36 to MX10, MX40 to MX11, MX44 to MX12, MX48 to MX13, MX2 to MX14, MX6 to MX15, MX10 to MX16, MX14 to MX17, MX22 to MX19, MX5 to MX2, MX26 to MX20, MX29 to MX21, MX33 to MX22, MX37 to MX23, MX41 to MX24, MX45 to MX25, MX49 to MX26, MX3 to MX27, MX7 to MX28, MX11 to MX29, MX9 to MX3, MX15 to MX30, MX19 to MX31, MX23 to MX32, MX27 to MX33, MX30 to MX34, MX34 to MX35, MX38 to MX36, MX42 to MX37, MX46 to MX38, MX50 to MX39, MX13 to MX4, MX4 to MX40, MX8 to MX41, MX12 to MX42, MX16 to MX43, MX20 to MX44, MX24 to MX45, MX31 to MX46, MX35 to MX47, MX39 to MX48, MX43 to MX49, MX17 to MX5, MX47 to MX50, MX21 to MX6, MX25 to MX7, MX28 to MX8, MX32 to MX9
Other:
- note removed: "1.0"
- note removed: "2020-02-15"
- note removed: "UT47 Nordic - Matrix"
