File: UT51.kicad_pcb (KiCad board)
At the start: 2 copper layers, 238.1 x 76.2 mm, 136 parts, among them SW1 SW_PUSH, U1 ATMEGA32U2-AU, U2 PRTR5V0U2X, Y1 16MHz

Commit message: Added the new coloumn
Added all the needed components, just need to fix the PCB.
Parts:
- removed the G*** at (265.1, 103.2) (x2)
- added D48: SOD-123, Diode_SMD:D_1206_3216Metric, F.Cu at (283.4, 39.7)
- added D49: SOD-123, Diode_SMD:D_1206_3216Metric, F.Cu at (270.7, 83.3)
- added D50: SOD-123, Diode_SMD:D_1206_3216Metric, F.Cu at (268.3, 64.3)
- added D51: SOD-123, Diode_SMD:D_1206_3216Metric, B.Cu at (272.3, 102.4)
- added MX48: MX-NoLED, footprints:Kailh_socket_MX, F.Cu at (274.6, 41.3)
- added MX49: MX-NoLED, footprints:Kailh_socket_MX, F.Cu at (279.4, 79.4)
- added MX50: MX-NoLED, footprints:Kailh_socket_MX, F.Cu at (277.0, 60.3)
- added MX51: MX-NoLED, footprints:Kailh_socket_MX, F.Cu at (279.4, 98.4)
- C1, C2, C3, C4, C5, C6, CR1, CR2, CR3, CR4, CR5, CR6, CR7, CR8: footprint Capacitors_SMD:C_0603 -> Capacitor_SMD:C_1206_3216Metric
- D1, D10, D11, D12, D13, D14, D15, D16, D17, D18, D19, D2, D20, D21, D22, D23, D24, D25, D26, D27, D28, D29, D3, D30, D31, D32, D33, D34, D35, D36, D37, D38, D39, D4, D40, D41, D42, D43, D44, D45, D46, D47, D5, D6, D7, D8, D9: footprint Diodes_SMD:D_SOD-123 -> Diode_SMD:D_1206_3216Metric
- F1: footprint Fuse_Holders_and_Fuses:Fuse_SMD1206_Reflow -> Fuse:Fuse_1206_3216Metric
- MX1, MX10, MX11, MX14, MX15, MX16, MX17, MX18, MX19, MX2, MX20, MX21, MX22, MX23, MX26, MX27, MX28, MX29, MX3, MX30, MX31, MX32, MX33, MX34, MX35, MX36, MX37, MX38, MX39, MX4, MX40, MX44, MX45, MX46, MX47, MX5, MX6, MX7, MX8, MX9: value MX-1U -> MX-NoLED; footprint MX_Alps_Hybrid:MXOnly-1U-Hotswap -> footprints:Kailh_socket_MX
- MX12, MX25: value MX-1.5U -> MX-NoLED; footprint MX_Alps_Hybrid:MXOnly-1.5U-Hotswap -> footprints:Kailh_socket_MX
- MX13, MX24, MX41, MX43: value MX-1.25U -> MX-NoLED; footprint MX_Alps_Hybrid:MXOnly-1.25U-Hotswap -> footprints:Kailh_socket_MX
- MX42: value MX-2U -> MX-NoLED; footprint MX_Alps_Hybrid:MXOnly-2U-Hotswap-ReversedStabilizers -> footprints:Kailh_socket_MX
- R1, R2, R3, R4, R5, R6: footprint Resistors_SMD:R_0603 -> Resistor_SMD:R_1206_3216Metric
- RGB1, RGB2, RGB3, RGB4, RGB5, RGB6, RGB7, RGB8: value VAL** -> WS2812B; footprint WS2812B:WS2812B -> LED_SMD:LED_WS2812B_PLCC4_5.0x5.0mm_P3.2mm
- SW1: value SW_PUSH -> SW_Push; footprint Molex-0548190589:SKQG-1155865 -> Button_Switch_SMD:SW_SPST_CK_RS282G05A3
- U1: footprint Housings_DFN_QFN:QFN-32-1EP_5x5mm_Pitch0.5mm -> Package_DFN_QFN:QFN-32-1EP_5x5mm_P0.5mm_EP3.1x3.1mm
- U2: footprint locallib:SOT143B -> Package_TO_SOT_SMD:SOT-143
- USB1: value HRO-TYPE-C-31-M-12 -> USB_C_Receptacle_USB2.0; footprint Type-C:HRO-TYPE-C-31-M-12-Assembly -> Connector_USB:USB_C_Receptacle_HRO_TYPE-C-31-M-12
- Y1: footprint Crystals:Crystal_SMD_3225-4pin_3.2x2.5mm -> Crystal:Crystal_SMD_0603-4Pin_6.0x3.5mm
- moved REF** 23.8 mm to (284.2, 50.8)
- moved REF** 19.0 mm to (279.4, 88.9)
- moved D47 15.9 mm to (268.3, 99.8)
- moved MX12 4.76 mm to (250.8, 41.3), turned to 0 degrees
- moved MX24 2.38 mm to (255.6, 60.3)
- turned RGB1 to 180 degrees
- turned RGB2 to 180 degrees
- turned RGB3 to 180 degrees
- turned RGB4 to 180 degrees
- turned RGB5 to 180 degrees
- turned RGB6 to 180 degrees
- turned RGB7 to 180 degrees
- turned RGB8 to 180 degrees
Connections:
- D10 pad 1: ROW0 -> ROW1
- D11 pad 1: ROW0 -> ROW2
- D12 pad 1: ROW0 -> ROW3
- D13 pad 1: ROW1 -> ROW0
- D15 pad 1: ROW1 -> ROW2
- D16 pad 1: ROW1 -> ROW3
- D17 pad 1: ROW1 -> ROW0
- D19 pad 1: ROW1 -> ROW2
- D2 pad 1: ROW0 -> ROW1
- D20 pad 1: ROW1 -> ROW3
- D21 pad 1: ROW1 -> ROW0
- D23 pad 1: ROW1 -> ROW2
- D24 pad 1: ROW1 -> ROW3
- D25 pad 1: ROW2 -> ROW0
- D26 pad 1: ROW2 -> ROW1
- D28 pad 1: ROW2 -> ROW0
- D29 pad 1: ROW2 -> ROW1
- D3 pad 1: ROW0 -> ROW2
- D31 pad 1: ROW2 -> ROW3
- D32 pad 1: ROW2 -> ROW0
- D33 pad 1: ROW2 -> ROW1
- D35 pad 1: ROW2 -> ROW3
- D36 pad 1: ROW2 -> ROW0
- D37 pad 1: ROW3 -> ROW1
- D38 pad 1: ROW3 -> ROW2
- D4 pad 1: ROW0 -> ROW3
- D40 pad 1: ROW3 -> ROW0
- D41 pad 1: ROW3 -> ROW1
- D42 pad 1: ROW3 -> ROW2
- D44 pad 1: ROW3 -> ROW0
- D45 pad 1: ROW3 -> ROW1
- D46 pad 1: ROW3 -> ROW2
- D6 pad 1: ROW0 -> ROW1
- D7 pad 1: ROW0 -> ROW2
- D8 pad 1: ROW0 -> ROW3
- MX10 pad 1: COL9 -> COL2
- MX11 pad 1: COL10 -> COL2
- MX12 pad 1: COL11 -> COL2
- MX13 pad 1: COL0 -> COL3
- MX14 pad 1: COL1 -> COL3
- MX15 pad 1: COL2 -> COL3
- MX18 pad 1: COL5 -> COL4
- MX19 pad 1: COL6 -> COL4
- MX2 pad 1: COL1 -> COL0
- MX20 pad 1: COL7 -> COL4
- MX21 pad 1: COL8 -> COL5
- MX22 pad 1: COL9 -> COL5
- MX23 pad 1: COL10 -> COL5
- MX24 pad 1: COL11 -> COL5
- MX25 pad 1: COL0 -> COL6
- MX26 pad 1: COL1 -> COL6
- MX27 pad 1: COL2 -> COL6
- MX28 pad 1: COL3 -> COL7
- MX29 pad 1: COL4 -> COL7
- MX3 pad 1: COL2 -> COL0
- MX30 pad 1: COL5 -> COL7
- MX31 pad 1: COL6 -> COL7
- MX32 pad 1: COL7 -> COL8
- MX34 pad 1: COL9 -> COL8
- MX35 pad 1: COL10 -> COL8
- MX36 pad 1: COL11 -> COL9
- MX37 pad 1: COL0 -> COL9
- MX38 pad 1: COL1 -> COL9
- MX39 pad 1: COL2 -> COL9
- MX4 pad 1: COL3 -> COL0
- MX40 pad 1: COL3 -> COL10
- MX41 pad 1: COL4 -> COL10
- MX42 pad 1: COL5 -> COL10
- MX43 pad 1: COL7 -> COL10
- MX44 pad 1: COL8 -> COL11
- MX45 pad 1: COL9 -> COL11
- MX46 pad 1: COL10 -> COL11
- MX5 pad 1: COL4 -> COL1
- MX6 pad 1: COL5 -> COL1
- MX7 pad 1: COL6 -> COL1
- MX8 pad 1: COL7 -> COL1
- MX9 pad 1: COL8 -> COL2
- R6 pad 1: Net-(R6-Pad1) -> GND
- R6 pad 2: GND -> Net-(R6-Pad2)
- U1 pad 33: (no net) -> GND
- U1 pad 5: Net-(U1-Pad5) -> COL12
Routing:
- net COL5: track 178.9 -> 209.9 mm
- net COL2: track 238.6 -> 266.8 mm
- net Net-(D23-Pad2): track 22.4 -> 0.00 mm
- net COL9: track 100.6 -> 121.6 mm
- net Net-(D47-Pad2): track 19.6 -> 0.00 mm
- net Net-(D11-Pad2): track 19.6 -> 0.00 mm
- net COL10: track 83.6 -> 100.8 mm
- net COL7: track 138.2 -> 155.4 mm
- net COL3: track 219.4 -> 236.6 mm
- net COL1: track 259.7 -> 276.9 mm
- net COL0: track 280.7 -> 297.9 mm
- net COL8: track 119.0 -> 136.2 mm
- net COL4: track 199.1 -> 216.3 mm
- net COL11: track 81.2 -> 94.1 mm
- net COL6: track 134.7 -> 147.6 mm
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Other:
- board size 238.1 x 76.2 mm -> 257.2 x 76.2 mm
- board text added: "20200215 | Credits to ai03's UT47.2"
- board text added: "UT51"
- board text added: "minimon.no"
- board text removed: "Distributed by Keyhive | 20181128 | Credits to 40percent.club's Gnap"
- board text removed: "UT47.2"
- board text removed: "kb.ai03.me"

Commit message: Finished first revision
Should be okay to order now
Parts:
- removed the D22 at (225.4, 60.3)
- removed the D48 at (283.4, 39.7)
- removed the D49 at (270.7, 83.3)
- removed G***: LOGO, locallib:Keyhive-Silk
- removed the MX24 at (255.6, 60.3)
- removed the MX36 at (260.4, 79.4)
- removed the MX46 at (241.3, 98.4)
- removed the MX47 at (260.4, 98.4)
- removed the REF** at (150.8, 69.8)
- removed the REF** at (41.3, 88.9)
- removed the REF** at (41.3, 50.8)
- removed the REF** at (284.2, 50.8)
- removed the REF** at (279.4, 88.9)
- added D13: SOD-123, Diode_SMD:D_SOD-123, B.Cu at (270.7, 49.9)
- added D24: SOD-123, Diode_SMD:D_SOD-123, B.Cu at (244.5, 60.6)
- added D26: SOD-123, Diode_SMD:D_SOD-123, B.Cu at (284.7, 63.0)
- added MX25: MX-NoLED, footprints:Kailh_socket_MX, F.Cu at (255.6, 60.3)
- added MX38: MX-NoLED, footprints:Kailh_socket_MX, F.Cu at (260.4, 79.4)
- added MX49: MX-NoLED, footprints:Kailh_socket_MX, F.Cu at (241.3, 98.4)
- added MX50: MX-NoLED, footprints:Kailh_socket_MX, F.Cu at (260.4, 98.4)
- added REF**: Stabilizer_MX_2u, footprints:Stabilizer_MX_2u, F.Cu at (150.7, 97.6)
- C1, C2: value 22p -> 0.1u; footprint Capacitor_SMD:C_1206_3216Metric -> Capacitor_SMD:C_0603_1608Metric
- C3: value 1uF -> 4.7u; footprint Capacitor_SMD:C_1206_3216Metric -> Capacitor_SMD:C_0603_1608Metric
- C4, C5: value 0.1u -> 22p; footprint Capacitor_SMD:C_1206_3216Metric -> Capacitor_SMD:C_0603_1608Metric
- C6: value 4.7u -> 1uF; footprint Capacitor_SMD:C_1206_3216Metric -> Capacitor_SMD:C_0603_1608Metric
- CR1, CR2, CR3, CR4, CR5, CR6, CR7, CR8: footprint Capacitor_SMD:C_1206_3216Metric -> Capacitor_SMD:C_0603_1608Metric
- D1, D10, D11, D12, D2, D23, D3, D4, D5, D51, D6, D7, D8, D9: footprint Diode_SMD:D_1206_3216Metric -> Diode_SMD:D_SOD-123
- D14: renamed from D13; footprint Diode_SMD:D_1206_3216Metric -> Diode_SMD:D_SOD-123
- D15: renamed from D14; footprint Diode_SMD:D_1206_3216Metric -> Diode_SMD:D_SOD-123
- D16: renamed from D15; footprint Diode_SMD:D_1206_3216Metric -> Diode_SMD:D_SOD-123
- D17: renamed from D16; footprint Diode_SMD:D_1206_3216Metric -> Diode_SMD:D_SOD-123
- D18: renamed from D17; footprint Diode_SMD:D_1206_3216Metric -> Diode_SMD:D_SOD-123
- D19: renamed from D18; footprint Diode_SMD:D_1206_3216Metric -> Diode_SMD:D_SOD-123
- D20: renamed from D19; footprint Diode_SMD:D_1206_3216Metric -> Diode_SMD:D_SOD-123
- D21: renamed from D20; footprint Diode_SMD:D_1206_3216Metric -> Diode_SMD:D_SOD-123
- D22: renamed from D21; footprint Diode_SMD:D_1206_3216Metric -> Diode_SMD:D_SOD-123
- D25: renamed from D24; footprint Diode_SMD:D_1206_3216Metric -> Diode_SMD:D_SOD-123
- D27: renamed from D25; footprint Diode_SMD:D_1206_3216Metric -> Diode_SMD:D_SOD-123
- D28: renamed from D26; footprint Diode_SMD:D_1206_3216Metric -> Diode_SMD:D_SOD-123
- D29: renamed from D27; footprint Diode_SMD:D_1206_3216Metric -> Diode_SMD:D_SOD-123
- D30: renamed from D28; footprint Diode_SMD:D_1206_3216Metric -> Diode_SMD:D_SOD-123
- D31: renamed from D29; footprint Diode_SMD:D_1206_3216Metric -> Diode_SMD:D_SOD-123
- D32: renamed from D30; footprint Diode_SMD:D_1206_3216Metric -> Diode_SMD:D_SOD-123
- D33: renamed from D31; footprint Diode_SMD:D_1206_3216Metric -> Diode_SMD:D_SOD-123
- D34: renamed from D32; footprint Diode_SMD:D_1206_3216Metric -> Diode_SMD:D_SOD-123
- D35: renamed from D33; footprint Diode_SMD:D_1206_3216Metric -> Diode_SMD:D_SOD-123
- D36: renamed from D34; footprint Diode_SMD:D_1206_3216Metric -> Diode_SMD:D_SOD-123
- D37: renamed from D35; footprint Diode_SMD:D_1206_3216Metric -> Diode_SMD:D_SOD-123
- D38: renamed from D36; footprint Diode_SMD:D_1206_3216Metric -> Diode_SMD:D_SOD-123
- D39: renamed from D50; footprint Diode_SMD:D_1206_3216Metric -> Diode_SMD:D_SOD-123; moved to B.Cu
- D40: renamed from D37; footprint Diode_SMD:D_1206_3216Metric -> Diode_SMD:D_SOD-123
- D41: renamed from D38; footprint Diode_SMD:D_1206_3216Metric -> Diode_SMD:D_SOD-123
- D42: renamed from D39; footprint Diode_SMD:D_1206_3216Metric -> Diode_SMD:D_SOD-123
- D43: renamed from D40; footprint Diode_SMD:D_1206_3216Metric -> Diode_SMD:D_SOD-123
- D44: renamed from D41; footprint Diode_SMD:D_1206_3216Metric -> Diode_SMD:D_SOD-123
- D45: renamed from D42; footprint Diode_SMD:D_1206_3216Metric -> Diode_SMD:D_SOD-123
- D46: renamed from D43; footprint Diode_SMD:D_1206_3216Metric -> Diode_SMD:D_SOD-123
- D47: renamed from D44; footprint Diode_SMD:D_1206_3216Metric -> Diode_SMD:D_SOD-123
- D48: renamed from D45; footprint Diode_SMD:D_1206_3216Metric -> Diode_SMD:D_SOD-123
- D49: renamed from D46; footprint Diode_SMD:D_1206_3216Metric -> Diode_SMD:D_SOD-123
- D50: renamed from D47; footprint Diode_SMD:D_1206_3216Metric -> Diode_SMD:D_SOD-123
- F1: footprint Fuse:Fuse_1206_3216Metric -> Fuse:Fuse_0603_1608Metric
- R1, R4: footprint Resistor_SMD:R_1206_3216Metric -> Resistor_SMD:R_0603_1608Metric
- R2: value 22 -> 10k; footprint Resistor_SMD:R_1206_3216Metric -> Resistor_SMD:R_0603_1608Metric
- R3: value 22 -> 5.1k; footprint Resistor_SMD:R_1206_3216Metric -> Resistor_SMD:R_0603_1608Metric
- R5: value 10k -> 22; footprint Resistor_SMD:R_1206_3216Metric -> Resistor_SMD:R_0603_1608Metric
- R6: value 5.1k -> 22; footprint Resistor_SMD:R_1206_3216Metric -> Resistor_SMD:R_0603_1608Metric
- U2: footprint Package_TO_SOT_SMD:SOT-143 -> footprints:SOT-143B
- Y1: footprint Crystal:Crystal_SMD_0603-4Pin_6.0x3.5mm -> Crystal:Crystal_SMD_3225-4Pin_3.2x2.5mm_HandSoldering
- moved SW1 71.8 mm to (281.7, 35.7)
- moved C3 34.0 mm to (269.8, 70.8), turned to 0 degrees
- moved R3 33.3 mm to (273.3, 34.5)
- moved R1 33.0 mm to (261.2, 44.0)
- moved C4 30.6 mm to (275.7, 63.9), turned to 0 degrees
- moved R5 29.8 mm to (266.2, 53.6)
- moved R6 27.4 mm to (266.2, 55.2), turned to 180 degrees
- moved F1 26.1 mm to (260.5, 41.5), turned to 90 degrees
- moved C5 25.9 mm to (275.7, 68.1)
- moved D39 25.4 mm to (285.2, 83.2), turned to 90 degrees
- moved D12 21.2 mm to (242.9, 43.9)
- moved CR8 20.7 mm to (271.5, 83.3)
- moved RGB8 20.7 mm to (271.5, 87.3)
- moved R4 20.1 mm to (273.3, 36.1), turned to 0 degrees
- moved Y1 19.8 mm to (270.7, 66.0)
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- renumbered MX48 to MX13, MX13 to MX14, MX14 to MX15, MX15 to MX16, MX16 to MX17, MX17 to MX18, MX18 to MX19, MX19 to MX20, MX20 to MX21, MX21 to MX22, MX22 to MX23, MX23 to MX24, MX50 to MX26, MX25 to MX27, MX26 to MX28, MX27 to MX29, MX28 to MX30, MX29 to MX31, MX30 to MX32, MX31 to MX33, MX32 to MX34, MX33 to MX35, MX34 to MX36, MX35 to MX37, MX49 to MX39, MX37 to MX40, MX38 to MX41, MX39 to MX42, MX40 to MX43, MX41 to MX44, MX42 to MX45, MX43 to MX46, MX44 to MX47, MX45 to MX48
Connections:
- C1 pad 1: Net-(C1-Pad1) -> +5V
- C2 pad 1: Net-(C2-Pad1) -> +5V
- C3 pad 1: Net-(C3-Pad1) -> +5V
- C4 pad 1: +5V -> Net-(C4-Pad1)
- C5 pad 1: +5V -> Net-(C5-Pad1)
- C6 pad 1: +5V -> Net-(C6-Pad1)
- D10 pad 1: ROW1 -> ROW0
- D11 pad 1: ROW2 -> ROW0
- D12 pad 1: ROW3 -> ROW0
- D14 pad 1: ROW0 -> ROW1
- D16 pad 1: ROW2 -> ROW1
- D17 pad 1: ROW3 -> ROW1
- D18 pad 1: ROW0 -> ROW1
- D2 pad 1: ROW1 -> ROW0
- D20 pad 1: ROW2 -> ROW1
- D21 pad 1: ROW3 -> ROW1
- D22 pad 1: ROW0 -> ROW1
- D23 pad 1: ROW2 -> ROW1
- D25 pad 1: ROW3 -> ROW1
- D27 pad 1: ROW0 -> ROW2
- D28 pad 1: ROW1 -> ROW2
- D3 pad 1: ROW2 -> ROW0
- D30 pad 1: ROW0 -> ROW2
- D31 pad 1: ROW1 -> ROW2
- D33 pad 1: ROW3 -> ROW2
- D34 pad 1: ROW0 -> ROW2
- D35 pad 1: ROW1 -> ROW2
- D37 pad 1: ROW3 -> ROW2
- D38 pad 1: ROW0 -> ROW2
- D39 pad 2: Net-(D50-Pad2) (its old number) -> Net-(D39-Pad2)
- D4 pad 1: ROW3 -> ROW0
- D40 pad 1: ROW1 -> ROW3
- D41 pad 1: ROW2 -> ROW3
- D43 pad 1: ROW0 -> ROW3
- D44 pad 1: ROW1 -> ROW3
- D45 pad 1: ROW2 -> ROW3
- D47 pad 1: ROW0 -> ROW3
- D48 pad 1: ROW1 -> ROW3
- D49 pad 1: ROW2 -> ROW3
- D6 pad 1: ROW1 -> ROW0
- D7 pad 1: ROW2 -> ROW0
- D8 pad 1: ROW3 -> ROW0
- MX10 pad 1: COL2 -> COL9
- MX11 pad 1: COL2 -> COL10
- MX12 pad 1: COL2 -> COL11
- MX14 pad 1: COL3 -> COL0
- MX15 pad 1: COL3 -> COL1
- MX16 pad 1: COL3 -> COL2
- MX19 pad 1: COL4 -> COL5
- MX2 pad 1: COL0 -> COL1
- MX20 pad 1: COL4 -> COL6
- MX21 pad 1: COL4 -> COL7
- MX22 pad 1: COL5 -> COL8
- MX23 pad 1: COL5 -> COL9
- MX23 pad 2: Net-(D22-Pad2) (its old number) -> Net-(D23-Pad2)
- MX24 pad 1: COL5 -> COL10
- MX24 pad 2: Net-(D23-Pad2) -> Net-(D24-Pad2)
- MX26 pad 2: Net-(D50-Pad2) (its old number) -> Net-(D26-Pad2)
- MX27 pad 1: COL6 -> COL0
- MX28 pad 1: COL6 -> COL1
- MX29 pad 1: COL6 -> COL2
- MX3 pad 1: COL0 -> COL2
- MX30 pad 1: COL7 -> COL3
- MX31 pad 1: COL7 -> COL4
- MX32 pad 1: COL7 -> COL5
- MX33 pad 1: COL7 -> COL6
- MX34 pad 1: COL8 -> COL7
- MX36 pad 1: COL8 -> COL9
- MX37 pad 1: COL8 -> COL10
- MX39 pad 2: Net-(D49-Pad2) (its old number) -> Net-(D39-Pad2)
- MX4 pad 1: COL0 -> COL3
- MX40 pad 1: COL9 -> COL0
- MX41 pad 1: COL9 -> COL1
- MX42 pad 1: COL9 -> COL2
- MX43 pad 1: COL10 -> COL3
- MX44 pad 1: COL10 -> COL4
- MX45 pad 1: COL10 -> COL5
- MX46 pad 1: COL10 -> COL7
- MX47 pad 1: COL11 -> COL8
- MX48 pad 1: COL11 -> COL9
- MX5 pad 1: COL1 -> COL4
- MX6 pad 1: COL1 -> COL5
- MX7 pad 1: COL1 -> COL6
- MX8 pad 1: COL1 -> COL7
- MX9 pad 1: COL2 -> COL8
- R2 pad 1: D- -> GND
- R3 pad 1: Net-(R3-Pad1) -> GND
- R3 pad 2: D+ -> Net-(R3-Pad2)
- R5 pad 1: GND -> D-
- R6 pad 1: GND -> Net-(R6-Pad1)
- R6 pad 2: Net-(R6-Pad2) -> D+
- U1 pad 1: Net-(C1-Pad1) -> Net-(C4-Pad1)
- U1 pad 13: Net-(R5-Pad2) -> Net-(R2-Pad2)
- U1 pad 2: Net-(C2-Pad1) -> Net-(C5-Pad1)
- U1 pad 27: Net-(C3-Pad1) -> Net-(C6-Pad1)
- U2 pad 2: Net-(R3-Pad1) -> Net-(R6-Pad1)
- U2 pad 3: Net-(R2-Pad2) -> Net-(R5-Pad2)
- USB1 pad A5: Net-(R6-Pad2) -> Net-(R3-Pad2)
- USB1 pad A6: Net-(R3-Pad1) -> Net-(R6-Pad1)
- USB1 pad A7: Net-(R2-Pad2) -> Net-(R5-Pad2)
- USB1 pad B6: Net-(R3-Pad1) -> Net-(R6-Pad1)
- USB1 pad B7: Net-(R2-Pad2) -> Net-(R5-Pad2)
- Y1 pad 1: Net-(C1-Pad1) -> Net-(C4-Pad1)
- Y1 pad 3: Net-(C2-Pad1) -> Net-(C5-Pad1)
Routing:
- net COL12: track 0.00 -> 70.9 mm, vias 0 -> 5
- net GND: track 663.5 -> 721.7 mm, vias 24 -> 19
- net ROW3: track 254.0 -> 283.2 mm
- net +5V: track 538.5 -> 562.9 mm, vias 6 -> 5
- net Net-(R6-Pad1): track 0.00 -> 21.9 mm
- net Net-(R3-Pad1): track 21.5 -> 0.00 mm, vias 2 -> 0
- net ROW2: track 237.1 -> 258.5 mm, vias 2 -> 0
- net Net-(D25-Pad2): track 4.30 -> 25.7 mm
- net Net-(RGB1-Pad2): track 64.1 -> 83.7 mm
- net Net-(D11-Pad2): track 0.00 -> 19.6 mm
- net Net-(R2-Pad2): track 25.3 -> 6.63 mm, vias 2 -> 0
- net Net-(RGB7-Pad2): track 66.4 -> 84.3 mm
- net Net-(R5-Pad2): track 2.75 -> 19.6 mm
- net ROW0: track 278.7 -> 263.0 mm, vias 4 -> 5
- net ROW1: track 264.6 -> 251.0 mm, vias 0 -> 2
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Other:
- board text added: "20200329 | Credits to ai03's UT47.2"
- board text removed: "20200215 | Credits to ai03's UT47.2"
