File: UT51.sch (KiCad schematic (older format))
At the start: 34 parts, among them SW1 SW_Push, U1 ATMEGA32U2-AU, U2 PRTR5V0U2X, Y1 16MHz

Commit message: Added the new coloumn
Added all the needed components, just need to fix the PCB.
Parts:
- C1, C2, C3, C4, C5, C6, CR1, CR2, CR3, CR4, CR5, CR6, CR7, CR8: footprint Capacitors_SMD:C_0603 -> Capacitor_SMD:C_1206_3216Metric
- F1: footprint Fuse_Holders_and_Fuses:Fuse_SMD1206_Reflow -> Fuse:Fuse_1206_3216Metric
- R1, R2, R3, R4, R5, R6: footprint Resistors_SMD:R_0603 -> Resistor_SMD:R_1206_3216Metric
- SW1: footprint Molex-0548190589:SKQG-1155865 -> Button_Switch_SMD:SW_SPST_CK_RS282G05A3
- U1: footprint Housings_DFN_QFN:QFN-32-1EP_5x5mm_Pitch0.5mm -> Package_DFN_QFN:QFN-32-1EP_5x5mm_P0.5mm_EP3.1x3.1mm
- USB1: footprint Type-C:HRO-TYPE-C-31-M-12-Assembly -> Connector_USB:USB_C_Receptacle_HRO_TYPE-C-31-M-12
- Y1: footprint Crystals:Crystal_SMD_3225-4pin_3.2x2.5mm -> Crystal:Crystal_SMD_0603-4Pin_6.0x3.5mm
- gave numbers to parts that had none: 7
Connections:
- no-connect marks 2 -> 6
Changed lines of the file:
@@
 F 0 "U1" H 3350 3000 50  0000 C CNN
 F 1 "ATMEGA32U2-AU" H 4100 1650 50  0000 C CNN
-F 2 "Housings_DFN_QFN:QFN-32-1EP_5x5mm_Pitch0.5mm" H 3200 3050 50  0001 C CNN
+F 2 "Package_DFN_QFN:QFN-32-1EP_5x5mm_P0.5mm_EP3.1x3.1mm" H 3200 3050 50  0001 C CNN
 F 3 "http://www.atmel.com/Images/doc7799.pdf" H 3450 1550 50  0001 C CNN
 	1    3350 3000
@@
 F 0 "Y1" V 1350 2350 50  0000 L CNN
 F 1 "16MHz" V 1500 2350 50  0000 L CNN
-F 2 "Crystals:Crystal_SMD_3225-4pin_3.2x2.5mm" H 1450 2200 50  0001 C CNN
+F 2 "Crystal:Crystal_SMD_0603-4Pin_6.0x3.5mm" H 1450 2200 50  0001 C CNN
 F 3 "~" H 1450 2200 50  0001 C CNN
 	1    1450 2200
@@
 F 0 "C1" V 1050 1925 50  0000 L CNN
 F 1 "22p" V 1050 2050 50  0000 L CNN
-F 2 "Capacitors_SMD:C_0603" H 1150 2000 50  0001 C CNN
+F 2 "Capacitor_SMD:C_1206_3216Metric" H 1150 2000 50  0001 C CNN
 F 3 "" H 1150 2000 50  0001 C CNN
 	1    1150 2000
@@
 F 0 "C2" V 1050 2325 50  0000 L CNN
 F 1 "22p" V 1050 2450 50  0000 L CNN
-F 2 "Capacitors_SMD:C_0603" H 1150 2400 50  0001 C CNN
+F 2 "Capacitor_SMD:C_1206_3216Metric" H 1150 2400 50  0001 C CNN
 F 3 "" H 1150 2400 50  0001 C CNN
 	1    1150 2400
@@
 F 0 "R1" V 2475 1925 50  0000 L CNN
 F 1 "10k" V 2475 1775 50  0000 L CNN
-F 2 "Resistors_SMD:R_0603" H 2400 1900 50  0001 C CNN
+F 2 "Resistor_SMD:R_1206_3216Metric" H 2400 1900 50  0001 C CNN
 F 3 "" H 2400 1900 50  0001 C CNN
 	1    2400 1900
@@
 F 0 "C3" V 2125 2675 50  0000 L CNN
 F 1 "1uF" V 2125 2800 50  0000 L CNN
-F 2 "Capacitors_SMD:C_0603" H 2250 2800 50  0001 C CNN
+F 2 "Capacitor_SMD:C_1206_3216Metric" H 2250 2800 50  0001 C CNN
 F 3 "" H 2250 2800 50  0001 C CNN
 	1    2250 2800
@@
 F 0 "R2" V 4025 5925 50  0000 L CNN
 F 1 "22" V 4025 6050 50  0000 L CNN
-F 2 "Resistors_SMD:R_0603" H 4100 6050 50  0001 C CNN
+F 2 "Resistor_SMD:R_1206_3216Metric" H 4100 6050 50  0001 C CNN
 F 3 "" H 4100 6050 50  0001 C CNN
 	1    4100 6050
@@
 F 0 "R3" V 4025 6025 50  0000 L CNN
 F 1 "22" V 4025 6150 50  0000 L CNN
-F 2 "Resistors_SMD:R_0603" H 4100 6150 50  0001 C CNN
+F 2 "Resistor_SMD:R_1206_3216Metric" H 4100 6150 50  0001 C CNN
 F 3 "" H 4100 6150 50  0001 C CNN
 	1    4100 6150
@@
 F 0 "F1" V 2475 5325 50  0000 C CNN
 F 1 "500mA" V 2475 5525 50  0000 C CNN
-F 2 "Fuse_Holders_and_Fuses:Fuse_SMD1206_Reflow" H 2600 5250 50  0001 L CNN
+F 2 "Fuse:Fuse_1206_3216Metric" H 2600 5250 50  0001 L CNN
 F 3 "" H 2550 5450 50  0001 C CNN
 	1    2550 5450
@@
 F 0 "R5" V 4700 4000 50  0000 L CNN
 F 1 "10k" V 4700 4125 50  0000 L CNN
-F 2 "Resistors_SMD:R_0603" H 4775 4100 50  0001 C CNN
+F 2 "Resistor_SMD:R_1206_3216Metric" H 4775 4100 50  0001 C CNN
 F 3 "" H 4775 4100 50  0001 C CNN
 	1    4775 4100
@@
 $EndComp
 $Comp
-L LED:WS2812B RGB?
+L LED:WS2812B RGB4
 U 1 1 59E67428
 P 10200 2300
-F 0 "RGB?" H 10000 2650 60  0000 C CNN
+F 0 "RGB4" H 10000 2650 60  0000 C CNN
 F 1 "WS2812B" H 10400 2650 60  0000 C CNN
 F 2 "LED_SMD:LED_WS2812B_PLCC4_5.0x5.0mm_P3.2mm" V 10150 2300 60  0001 C CNN
@@
 F 0 "CR1" H 6460 945 50  0000 L CNN
 F 1 "0.1u" H 6460 795 50  0000 L CNN
-F 2 "Capacitors_SMD:C_0603" H 6450 875 50  0001 C CNN
+F 2 "Capacitor_SMD:C_1206_3216Metric" H 6450 875 50  0001 C CNN
 F 3 "" H 6450 875 50  0001 C CNN
 	1    6450 875
@@
 F 0 "CR2" H 6660 945 50  0000 L CNN
 F 1 "0.1u" H 6660 795 50  0000 L CNN
-F 2 "Capacitors_SMD:C_0603" H 6650 875 50  0001 C CNN
+F 2 "Capacitor_SMD:C_1206_3216Metric" H 6650 875 50  0001 C CNN
 F 3 "" H 6650 875 50  0001 C CNN
 	1    6650 875
@@
 F 0 "CR3" H 6860 945 50  0000 L CNN
 F 1 "0.1u" H 6860 795 50  0000 L CNN
-F 2 "Capacitors_SMD:C_0603" H 6850 875 50  0001 C CNN
+F 2 "Capacitor_SMD:C_1206_3216Metric" H 6850 875 50  0001 C CNN
 F 3 "" H 6850 875 50  0001 C CNN
 	1    6850 875
@@
 F 0 "CR4" H 7060 945 50  0000 L CNN
 F 1 "0.1u" H 7060 795 50  0000 L CNN
-F 2 "Capacitors_SMD:C_0603" H 7050 875 50  0001 C CNN
+F 2 "Capacitor_SMD:C_1206_3216Metric" H 7050 875 50  0001 C CNN
 F 3 "" H 7050 875 50  0001 C CNN
 	1    7050 875
@@
 F 0 "CR5" H 7260 945 50  0000 L CNN
 F 1 "0.1u" H 7260 795 50  0000 L CNN
-F 2 "Capacitors_SMD:C_0603" H 7250 875 50  0001 C CNN
+F 2 "Capacitor_SMD:C_1206_3216Metric" H 7250 875 50  0001 C CNN
 F 3 "" H 7250 875 50  0001 C CNN
 	1    7250 875
@@
 F 0 "CR6" H 7460 945 50  0000 L CNN
 F 1 "0.1u" H 7460 795 50  0000 L CNN
-F 2 "Capacitors_SMD:C_0603" H 7450 875 50  0001 C CNN
+F 2 "Capacitor_SMD:C_1206_3216Metric" H 7450 875 50  0001 C CNN
 F 3 "" H 7450 875 50  0001 C CNN
 	1    7450 875
@@
 F 0 "CR7" H 7660 945 50  0000 L CNN
 F 1 "0.1u" H 7660 795 50  0000 L CNN
-F 2 "Capacitors_SMD:C_0603" H 7650 875 50  0001 C CNN
+F 2 "Capacitor_SMD:C_1206_3216Metric" H 7650 875 50  0001 C CNN
 F 3 "" H 7650 875 50  0001 C CNN
 	1    7650 875
@@
 F 0 "CR8" H 6560 1420 50  0000 L CNN
 F 1 "0.1u" H 6560 1270 50  0000 L CNN
-F 2 "Capacitors_SMD:C_0603" H 6550 1350 50  0001 C CNN
+F 2 "Capacitor_SMD:C_1206_3216Metric" H 6550 1350 50  0001 C CNN
 F 3 "" H 6550 1350 50  0001 C CNN
 	1    6550 1350
@@
 F 0 "C4" H 1010 970 50  0000 L CNN
 F 1 "0.1u" H 1010 820 50  0000 L CNN
-F 2 "Capacitors_SMD:C_0603" H 1000 900 50  0001 C CNN
+F 2 "Capacitor_SMD:C_1206_3216Metric" H 1000 900 50  0001 C CNN
 F 3 "" H 1000 900 50  0001 C CNN
 	1    1000 900
@@
 F 0 "C5" H 1210 970 50  0000 L CNN
 F 1 "0.1u" H 1210 820 50  0000 L CNN
-F 2 "Capacitors_SMD:C_0603" H 1200 900 50  0001 C CNN
+F 2 "Capacitor_SMD:C_1206_3216Metric" H 1200 900 50  0001 C CNN
 F 3 "" H 1200 900 50  0001 C CNN
 	1    1200 900
@@
 F 0 "C6" H 1410 970 50  0000 L CNN
 F 1 "4.7u" H 1410 820 50  0000 L CNN
-F 2 "Capacitors_SMD:C_0603" H 1400 900 50  0001 C CNN
+F 2 "Capacitor_SMD:C_1206_3216Metric" H 1400 900 50  0001 C CNN
 F 3 "" H 1400 900 50  0001 C CNN
 	1    1400 900
@@
 F 0 "SW1" H 2450 1710 50  0000 C CNN
 F 1 "SW_Push" H 2300 1520 50  0000 C CNN
-F 2 "Molex-0548190589:SKQG-1155865" H 2300 1600 60  0001 C CNN
+F 2 "Button_Switch_SMD:SW_SPST_CK_RS282G05A3" H 2300 1600 60  0001 C CNN
 F 3 "~" H 2300 1600 60  0000 C CNN
 	1    2300 1600
@@
 F 0 "USB1" H 1500 6950 60  0000 C CNN
 F 1 "USB_C_Receptacle_USB2.0" H 1500 6850 60  0000 C CNN
-F 2 "Type-C:HRO-TYPE-C-31-M-12-Assembly" H 1500 6050 60  0001 C CNN
+F 2 "Connector_USB:USB_C_Receptacle_HRO_TYPE-C-31-M-12" H 1500 6050 60  0001 C CNN
 F 3 "https://www.usb.org/sites/default/files/documents/usb_type-c.zip" H 1500 6050 60  0001 C CNN
 	1    1500 6050
@@
 F 0 "R4" V 2125 5625 50  0000 L CNN
 F 1 "5.1k" V 2125 5750 50  0000 L CNN
-F 2 "Resistors_SMD:R_0603" H 2200 5750 50  0001 C CNN
+F 2 "Resistor_SMD:R_1206_3216Metric" H 2200 5750 50  0001 C CNN
 F 3 "" H 2200 5750 50  0001 C CNN
 	1    2200 5750
@@
 F 0 "R6" V 2125 5525 50  0000 L CNN
 F 1 "5.1k" V 2125 5650 50  0000 L CNN
-F 2 "Resistors_SMD:R_0603" H 2200 5650 50  0001 C CNN
+F 2 "Resistor_SMD:R_1206_3216Metric" H 2200 5650 50  0001 C CNN
 F 3 "" H 2200 5650 50  0001 C CNN
 	1    2200 5650
@@
 COL12
 $Comp
-L power:GND #PWR?
+L power:GND #PWR02
 U 1 1 5E4BB8E0
 P 3250 4650
-F 0 "#PWR?" H 3250 4400 50  0001 C CNN
+F 0 "#PWR02" H 3250 4400 50  0001 C CNN
 F 1 "GND" H 3250 4500 50  0000 C CNN
 F 2 "" H 3250 4650 50  0001 C CNN
@@
 	3250 4400 3250 4650
 $Comp
-L power:+5V #PWR?
+L power:+5V #PWR07
 U 1 1 5E4F14D0
 P 3450 1500
-F 0 "#PWR?" H 3450 1350 50  0001 C CNN
+F 0 "#PWR07" H 3450 1350 50  0001 C CNN
 F 1 "+5V" V 3450 1700 50  0000 C CNN
 F 2 "" H 3450 1500 50  0001 C CNN
@@
 $EndComp
 $Comp
-L power:+5V #PWR?
+L power:+5V #PWR06
 U 1 1 5E4F1B09
 P 3350 1450
-F 0 "#PWR?" H 3350 1300 50  0001 C CNN
+F 0 "#PWR06" H 3350 1300 50  0001 C CNN
 F 1 "+5V" V 3350 1650 50  0000 C CNN
 F 2 "" H 3350 1450 50  0001 C CNN
@@
 $EndComp
 $Comp
-L LED:WS2812B RGB?
+L LED:WS2812B RGB2
 U 1 1 5E5E7D2D
 P 8400 2300
-F 0 "RGB?" H 8200 2650 60  0000 C CNN
+F 0 "RGB2" H 8200 2650 60  0000 C CNN
 F 1 "WS2812B" H 8600 2650 60  0000 C CNN
 F 2 "LED_SMD:LED_WS2812B_PLCC4_5.0x5.0mm_P3.2mm" V 8350 2300 60  0001 C CNN
@@
 $EndComp
 $Comp
-L LED:WS2812B RGB?
+L LED:WS2812B RGB3
 U 1 1 5E5E850D
 P 9300 2300
-F 0 "RGB?" H 9100 2650 60  0000 C CNN
+F 0 "RGB3" H 9100 2650 60  0000 C CNN
 F 1 "WS2812B" H 9500 2650 60  0000 C CNN
 F 2 "LED_SMD:LED_WS2812B_PLCC4_5.0x5.0mm_P3.2mm" V 9250 2300 60  0001 C CNN
@@
 $EndComp
 $Comp
-L LED:WS2812B RGB?
+L LED:WS2812B RGB5
 U 1 1 5E5EE103
 P 7500 3200
-F 0 "RGB?" H 7300 3550 60  0000 C CNN
+F 0 "RGB5" H 7300 3550 60  0000 C CNN
 F 1 "WS2812B" H 7700 3550 60  0000 C CNN
 F 2 "LED_SMD:LED_WS2812B_PLCC4_5.0x5.0mm_P3.2mm" V 7450 3200 60  0001 C CNN
@@
 $EndComp
 $Comp
-L LED:WS2812B RGB?
+L LED:WS2812B RGB6
 U 1 1 5E5EF191
 P 8400 3200
-F 0 "RGB?" H 8200 3550 60  0000 C CNN
+F 0 "RGB6" H 8200 3550 60  0000 C CNN
 F 1 "WS2812B" H 8600 3550 60  0000 C CNN
 F 2 "LED_SMD:LED_WS2812B_PLCC4_5.0x5.0mm_P3.2mm" V 8350 3200 60  0001 C CNN
@@
 $EndComp
 $Comp
-L LED:WS2812B RGB?
+L LED:WS2812B RGB7
 U 1 1 5E5EFA3D
 P 9300 3200
-F 0 "RGB?" H 9100 3550 60  0000 C CNN
+F 0 "RGB7" H 9100 3550 60  0000 C CNN
 F 1 "WS2812B" H 9500 3550 60  0000 C CNN
 F 2 "LED_SMD:LED_WS2812B_PLCC4_5.0x5.0mm_P3.2mm" V 9250 3200 60  0001 C CNN
@@
 $EndComp
 $Comp
-L LED:WS2812B RGB?
+L LED:WS2812B RGB8
 U 1 1 5E5F0102
 P 10200 3200
-F 0 "RGB?" H 10000 3550 60  0000 C CNN
+F 0 "RGB8" H 10000 3550 60  0000 C CNN
 F 1 "WS2812B" H 10400 3550 60  0000 C CNN
 F 2 "LED_SMD:LED_WS2812B_PLCC4_5.0x5.0mm_P3.2mm" V 10150 3200 60  0001 C CNN
@@
 Wire Wire Line
 	2950 6150 4000 6150
+NoConn ~ 10500 3200
+NoConn ~ 4050 3400
+NoConn ~ 4050 3200
+NoConn ~ -5050 -950
 $EndSCHEMATC

Commit message: Finished first revision
Should be okay to order now
Parts:
- C1: renamed from C4; footprint Capacitor_SMD:C_1206_3216Metric -> Capacitor_SMD:C_0603_1608Metric
- C2: renamed from C5; footprint Capacitor_SMD:C_1206_3216Metric -> Capacitor_SMD:C_0603_1608Metric
- C3: renamed from C6; footprint Capacitor_SMD:C_1206_3216Metric -> Capacitor_SMD:C_0603_1608Metric
- C4: renamed from C1; footprint Capacitor_SMD:C_1206_3216Metric -> Capacitor_SMD:C_0603_1608Metric
- C5: renamed from C2; footprint Capacitor_SMD:C_1206_3216Metric -> Capacitor_SMD:C_0603_1608Metric
- C6: renamed from C3; footprint Capacitor_SMD:C_1206_3216Metric -> Capacitor_SMD:C_0603_1608Metric
- CR1, CR2, CR3, CR4, CR5, CR6, CR7, CR8: footprint Capacitor_SMD:C_1206_3216Metric -> Capacitor_SMD:C_0603_1608Metric
- F1: footprint Fuse:Fuse_1206_3216Metric -> Fuse:Fuse_0603_1608Metric
- R1, R4: footprint Resistor_SMD:R_1206_3216Metric -> Resistor_SMD:R_0603_1608Metric
- R2: renamed from R5; footprint Resistor_SMD:R_1206_3216Metric -> Resistor_SMD:R_0603_1608Metric
- R3: renamed from R6; footprint Resistor_SMD:R_1206_3216Metric -> Resistor_SMD:R_0603_1608Metric
- R5: renamed from R2; footprint Resistor_SMD:R_1206_3216Metric -> Resistor_SMD:R_0603_1608Metric
- R6: renamed from R3; footprint Resistor_SMD:R_1206_3216Metric -> Resistor_SMD:R_0603_1608Metric
- U2: footprint Package_TO_SOT_SMD:SOT-143 -> footprints:SOT-143B
- Y1: footprint Crystal:Crystal_SMD_0603-4Pin_6.0x3.5mm -> Crystal:Crystal_SMD_3225-4Pin_3.2x2.5mm_HandSoldering
Connections:
- no-connect marks 6 -> 5
Other:
- note removed: "1.0"
- note removed: "2020-02-15"
- note removed: "UT47 Nordic"
